Commit message: adds minor Gazebo-related modifications

File: create_description/urdf/create_gazebo.urdf.xacro (robot description, xacro)
@@ -3,5 +3,5 @@
 	<xacro:macro name="sim_create">
 	  <gazebo>
-	    <controller:gazebo_ros_create name="create_controller" plugin="libgazebo_ros_create.so">
+	    <plugin name="create_controller" filename="libgazebo_ros_create.so">
 	      <alwaysOn>true</alwaysOn>
 	      <node_namespace>turtlebot_node</node_namespace>
@@ -15,5 +15,5 @@
 	      <updateRate>40</updateRate>
 	      <torque>1.0</torque>
-	    </controller:gazebo_ros_create>
+	    </plugin>
 	  </gazebo>
     <gazebo reference="left_wheel_link">
@@ -22,5 +22,5 @@
       <kp value="100000000.0"/>
       <kd value="10000.0"/>
-      <fdir value="1 0 0"/>
+      <fdir1 value="1 0 0"/>
     </gazebo>
     <gazebo reference="right_wheel_link">
@@ -29,5 +29,5 @@
       <kp value="100000000.0"/>
       <kd value="10000.0"/>
-      <fdir value="1 0 0"/>
+      <fdir1 value="1 0 0"/>
     </gazebo>
     <gazebo reference="rear_wheel_link">
@@ -46,110 +46,164 @@
 	<xacro:macro name="sim_imu">
 	  <gazebo>
-	    <controller:gazebo_ros_imu name="imu_controller" plugin="libgazebo_ros_imu.so">
+	    <plugin name="imu_controller" filename="libgazebo_ros_imu.so">
 	      <alwaysOn>true</alwaysOn>
 	      <updateRate>30</updateRate>
 	      <bodyName>gyro_link</bodyName>
 	      <topicName>imu/data</topicName>
-	      <serviceName>imu/service</serviceName>
 	      <gaussianNoise>${0.0017*0.0017}</gaussianNoise>
-	      <xyzOffset>0 0 0</xyzOffset>
-	      <rpyOffset>0 0 0</rpyOffset>
-	      <interface:position name="imu_position"/>
-	    </controller:gazebo_ros_imu>
+        <xyzOffsets>0 0 0</xyzOffsets>
+        <rpyOffsets>0 0 0</rpyOffsets>
+      </plugin>
 	  </gazebo>
 	</xacro:macro>
 	<xacro:macro name="sim_create_wall_sensor">
 	  <gazebo reference="wall_sensor_link">
-	    <sensor:ray name="wall_sensor">
-	      <alwaysActive>true</alwaysActive>
-	      <rayCount>1</rayCount>
-	      <rangeCount>1</rangeCount>
-	      <resRange>0.1</resRange>
-	      <minAngle>0</minAngle>
-	      <maxAngle>0</maxAngle>
-	      <minRange>0.0160</minRange>
-	      <maxRange>0.04</maxRange>
-	      <displayRays>false</displayRays>
-	    </sensor:ray>
+      <sensor type="ray" name="wall_sensor">
+        <always_on>true</always_on>
+        <update_rate>20.0</update_rate>
+        <pose>0 0 0 0 0 0</pose>
+        <visualize>false</visualize>
+        <ray>
+          <scan>
+            <horizontal>
+              <samples>1</samples>
+              <resolution>1</resolution>
+              <min_angle>0</min_angle>
+              <max_angle>0</max_angle>
+            </horizontal>
+          </scan>
+          <range>
+            <min>0.0160</min>
+            <max>0.04</max>
+            <resolution>0.1</resolution>
+          </range>
+        </ray>
+      </sensor>
 	  </gazebo>
 	</xacro:macro>
 	<xacro:macro name="sim_create_cliff_sensors">
 	  <gazebo reference="left_cliff_sensor_link">
-	    <sensor:ray name="left_cliff_sensor">
-	      <alwaysActive>true</alwaysActive>
-	      <rayCount>1</rayCount>
-	      <rangeCount>1</rangeCount>
-	      <resRange>0.1</resRange>
-	      <minAngle>0</minAngle>
-	      <maxAngle>0</maxAngle>
-	      <minRange>0.01</minRange>
-	      <maxRange>0.04</maxRange>
-	      <displayRays>false</displayRays>
-	    </sensor:ray>
+      <sensor type="ray" name="left_cliff_sensor">
+        <always_on>true</always_on>
+        <update_rate>20.0</update_rate>
+        <pose>0 0 0 0 0 0</pose>
+        <visualize>false</visualize>
+        <ray>
+          <scan>
+            <horizontal>
+              <samples>1</samples>
+              <resolution>1</resolution>
+              <min_angle>0</min_angle>
+              <max_angle>0</max_angle>
+            </horizontal>
+          </scan>
+          <range>
+            <min>0.01</min>
+            <max>0.04</max>
+            <resolution>0.1</resolution>
+          </range>
+        </ray>
+      </sensor>
 	  </gazebo>
 	  <gazebo reference="right_cliff_sensor_link">
-	    <sensor:ray name="right_cliff_sensor">
-	      <alwaysActive>true</alwaysActive>
-	      <rayCount>1</rayCount>
-	      <rangeCount>1</rangeCount>
-	      <resRange>0.1</resRange>
-	      <minAngle>0</minAngle>
-	      <maxAngle>0</maxAngle>
-	      <minRange>0.01</minRange>
-	      <maxRange>0.04</maxRange>
-	      <displayRays>false</displayRays>
-	    </sensor:ray>
+      <sensor type="ray" name="right_cliff_sensor">
+        <always_on>true</always_on>
+        <update_rate>20.0</update_rate>
+        <pose>0 0 0 0 0 0</pose>
+        <visualize>false</visualize>
+        <ray>
+          <scan>
+            <horizontal>
+              <samples>1</samples>
+              <resolution>1</resolution>
+              <min_angle>0</min_angle>
+              <max_angle>0</max_angle>
+            </horizontal>
+          </scan>
+          <range>
+            <min>0.01</min>
+            <max>0.04</max>
+            <resolution>0.1</resolution>
+          </range>
+        </ray>
+      </sensor>
 	  </gazebo>
 	  <gazebo reference="leftfront_cliff_sensor_link">
-	    <sensor:ray name="leftfront_cliff_sensor">
-	      <alwaysActive>true</alwaysActive>
-	      <rayCount>1</rayCount>
-	      <rangeCount>1</rangeCount>
-	      <resRange>0.1</resRange>
-	      <minAngle>0</minAngle>
-	      <maxAngle>0</maxAngle>
-	      <minRange>0.01</minRange>
-	      <maxRange>0.04</maxRange>
-	      <displayRays>false</displayRays>
-	    </sensor:ray>
+      <sensor type="ray" name="leftfront_cliff_sensor">
+        <always_on>true</always_on>
+        <update_rate>20.0</update_rate>
+        <pose>0 0 0 0 0 0</pose>
+        <visualize>false</visualize>
+        <ray>
+          <scan>
+            <horizontal>
+              <samples>1</samples>
+              <resolution>1</resolution>
+              <min_angle>0</min_angle>
+              <max_angle>0</max_angle>
+            </horizontal>
+          </scan>
+          <range>
+            <min>0.01</min>
+            <max>0.04</max>
+            <resolution>0.1</resolution>
+          </range>
+        </ray>
+      </sensor>
 	  </gazebo>
 	  <gazebo reference="rightfront_cliff_sensor_link">
-	    <sensor:ray name="rightfront_cliff_sensor">
-	      <alwaysActive>true</alwaysActive>
-	      <rayCount>1</rayCount>
-	      <rangeCount>1</rangeCount>
-	      <resRange>0.1</resRange>
-	      <minAngle>0</minAngle>
-	      <maxAngle>0</maxAngle>
-	      <minRange>0.01</minRange>
-	      <maxRange>0.04</maxRange>
-	      <displayRays>fan</displayRays>
-	    </sensor:ray>
+      <sensor type="ray" name="rightfront_cliff_sensor">
+        <always_on>true</always_on>
+        <update_rate>20.0</update_rate>
+        <pose>0 0 0 0 0 0</pose>
+        <visualize>false</visualize>
+        <ray>
+          <scan>
+            <horizontal>
+              <samples>1</samples>
+              <resolution>1</resolution>
+              <min_angle>0</min_angle>
+              <max_angle>0</max_angle>
+            </horizontal>
+          </scan>
+          <range>
+            <min>0.01</min>
+            <max>0.04</max>
+            <resolution>0.1</resolution>
+          </range>
+        </ray>
+      </sensor>
 	  </gazebo>
 	</xacro:macro>
 	<xacro:macro name="sim_laser">
 	  <gazebo reference="laser">
-	    <sensor:ray name="laser">
-	      <rayCount>180</rayCount>
-	      <rangeCount>180</rangeCount>
-	      <laserCount>1</laserCount>
-	      <origin>0.0 0.0 0.0</origin>
-	      <displayRays>false</displayRays>
-	      <minAngle>-130</minAngle>
-	      <maxAngle>130</maxAngle>
-	      <minRange>0.08</minRange>
-	      <maxRange>10.0</maxRange>
-	      <resRange>0.01</resRange>
-	      <updateRate>20</updateRate>
-	      <controller:gazebo_ros_laser name="gazebo_ros_laser_controller" plugin="libgazebo_ros_laser.so">
-	        <gaussianNoise>0.005</gaussianNoise>
-	        <alwaysOn>true</alwaysOn>
-	        <updateRate>20</updateRate>
-	        <topicName>scan</topicName>
-	        <frameName>laser</frameName>
-	        <interface:laser name="gazebo_ros_laser_iface" />
-	        <hokuyoMinIntensity>101.0</hokuyoMinIntensity>
-	      </controller:gazebo_ros_laser>
-	    </sensor:ray>
+      <sensor type="ray" name="laser">
+        <always_on>true</always_on>
+        <update_rate>20.0</update_rate>
+        <pose>0 0 0 0 0 0</pose>
+        <visualize>false</visualize>
+        <ray>
+          <scan>
+            <horizontal>
+              <samples>180</samples>
+              <resolution>1</resolution>
+              <min_angle>${-130.0*M_PI/180.0}</min_angle>
+              <max_angle>${130.0*M_PI/180.0}</max_angle>
+            </horizontal>
+          </scan>
+          <range>
+            <min>0.08</min>
+            <max>10.0</max>
+            <resolution>0.01</resolution>
+          </range>
+        </ray>
+        <plugin name="gazebo_ros_laser_controller" filename="libgazebo_ros_laser.so">
+          <gaussianNoise>0.005</gaussianNoise>
+          <alwaysOn>true</alwaysOn>
+          <updateRate>20</updateRate>
+          <topicName>scan</topicName>
+          <frameName>laser</frameName>
+        </plugin>
+      </sensor>
 	  </gazebo>
   </xacro:macro>
