Commit message: adds files formerly located at turtlebot_description

File: create_description/urdf/create.urdf.xacro (robot description, xacro)
@@ -1,273 +1,275 @@
 <?xml version="1.0"?>
-<robot name="turtlebot_hardware" xmlns:xacro="http://ros.org/wiki/xacro">
+<robot name="turtlebot_hardware"
+       xmlns:xacro="http://ros.org/wiki/xacro">
   <property name="M_PI" value="3.14159"/>
   <property name="SCALE" value="0.0254"/>
   <!-- Macro for TurtleBot body. Including Gazebo extensions, but does not include Kinect -->
-  <include filename="$(find turtlebot_description)/urdf/gazebo.urdf.xacro"/>
+  <include filename="$(find create_description)/urdf/create_gazebo.urdf.xacro"/>
   <property name="base_x" value="0.33" />
   <property name="base_y" value="0.33" />
-  <xacro:macro name="create">
-    <material name="Green">
-      <color rgba="0.0 0.8 0.0 1.0"/>
-    </material>
-  <!-- base_footprint is a fictitious link(frame) that is on the ground right below base_link origin, navigation stack depends on this frame -->
-  <link name="base_footprint">
-<!--
-    <inertial>
-      <mass value="0.0001" />
-      <origin xyz="0 0 0" />
-      <inertia ixx="0.0001" ixy="0.0" ixz="0.0"
-              iyy="0.0001" iyz="0.0"
-              izz="0.0001" />
-    </inertial>
--->
-    <visual>
-      <origin xyz="0 0 0" rpy="0 0 0" />
-      <geometry>
-        <box size="0.001 0.001 0.001" />
-      </geometry>
-      <material name="Green" />
-    </visual>
-    <collision>
-      <origin xyz="0 0 0.017" rpy="0 0 0" />
-      <geometry>
-       <box size="0.001 0.001 0.001" />
-      </geometry>
-    </collision>
-  </link>
-  <link name="base_link">
-    <inertial>
-      <mass value="2" />
-      <origin xyz="0 0 0.0" />
-      <inertia ixx="0.01" ixy="0.0" ixz="0.0"
-        iyy="0.01" iyz="0.0" izz="0.5" />
-    </inertial>
-    <visual>
-      <origin xyz=" 0 0 0.0308" rpy="0 0 0" />
-      <geometry>
-        <mesh filename="package://turtlebot_description/meshes/base/create_body.dae"/>
-      </geometry>
-    </visual>
-    <collision>
-      <origin xyz="0.0 0.0 0.0308" rpy="0 0 0" />
-      <geometry>
-        <cylinder length="0.0611632" radius="0.016495"/>
-      </geometry>
-    </collision>
-  </link>
-  <link name="wall_sensor_link">
-    <inertial>
-      <mass value="0.01" />
-      <origin xyz="0 0 0"/>
-      <inertia ixx="0.001" ixy="0.0" ixz="0.0"
-        iyy="0.001" iyz="0.0" izz="0.001" />
-    </inertial>
-  </link>
-  <link name="left_cliff_sensor_link">
-    <inertial>
-      <mass value="0.01" />
-      <origin xyz="0 0 0"/>
-      <inertia ixx="0.001" ixy="0.0" ixz="0.0"
-        iyy="0.001" iyz="0.0" izz="0.001" />
-    </inertial>
-  </link>
-  <link name="right_cliff_sensor_link">
-    <inertial>
-      <mass value="0.01" />
-      <origin xyz="0 0 0"/>
-      <inertia ixx="0.001" ixy="0.0" ixz="0.0"
-        iyy="0.001" iyz="0.0" izz="0.001" />
-    </inertial>
-  </link>
-  <link name="leftfront_cliff_sensor_link">
-    <inertial>
-      <mass value="0.01" />
-      <origin xyz="0 0 0"/>
-      <inertia ixx="1.0" ixy="0.0" ixz="0.0"
-        iyy="0.01" iyz="0.0" izz="0.01" />
-    </inertial>
-  </link>
-  <link name="rightfront_cliff_sensor_link">
-    <inertial>
-      <mass value="0.01" />
-      <origin xyz="0 0 0"/>
-      <inertia ixx="0.001" ixy="0.0" ixz="0.0"
-        iyy="0.001" iyz="0.0" izz="0.001" />
-    </inertial>
-  </link>
-  <joint name="base_footprint_joint" type="fixed">
-    <origin xyz="0 0 0.017" rpy="0 0 0" />
-    <parent link="base_footprint"/>
-    <child link="base_link" />
-  </joint>
-  <joint name="base_wall_sensor_joint" type="fixed">
-    <origin xyz="0.09 -0.120 0.042" rpy="0 0 -1.0" />
-    <parent link="base_link"/>
-    <child link="wall_sensor_link" />
-  </joint>
-  <joint name="base_left_cliff_sensor_joint" type="fixed">
-    <origin xyz="0.07 0.14 0.01" rpy="0 1.57079 0" />
-    <parent link="base_link"/>
-    <child link="left_cliff_sensor_link" />
-  </joint>
-  <joint name="base_right_cliff_sensor_joint" type="fixed">
-    <origin xyz="0.07 -0.14 0.01" rpy="0 1.57079 0" />
-    <parent link="base_link"/>
-    <child link="right_cliff_sensor_link" />
-  </joint>
-  <joint name="base_leftfront_cliff_sensor_joint" type="fixed">
-    <origin xyz="0.15 0.04 0.01" rpy="0 1.57079 0" />
-    <parent link="base_link"/>
-    <child link="leftfront_cliff_sensor_link" />
-  </joint>
-  <joint name="base_rightfront_cliff_sensor_joint" type="fixed">
-    <origin xyz="0.15 -0.04 0.01" rpy="0 1.57079 0" />
-    <parent link="base_link"/>
-    <child link="rightfront_cliff_sensor_link" />
-  </joint>
-  <link name="left_wheel_link">
-    <inertial>
-      <origin xyz="0 0 0"/>
-      <mass value="0.01" />
-      <inertia ixx="0.001" ixy="0.0" ixz="0.0"
-        iyy="0.001" iyz="0.0" izz="0.001" />
-    </inertial>
-    <visual>
-      <origin xyz="0 0 0" rpy="0 1.5707 1.5707" />
-      <geometry>
-        <cylinder radius="0.033" length = "0.023"/>
-      </geometry>
-    </visual>
-    <collision>
-      <origin xyz="0 0 0" rpy="0 1.5707 1.5707" />
-      <geometry>
-        <cylinder radius="0.033" length = "0.023"/>
-      </geometry>
-    </collision>
-  </link>
-  <joint name="left_wheel_joint" type="continuous">
-    <origin xyz="0 0.13 0.015" rpy="0 0 0"/>
-    <parent link="base_link"/>
-    <child link="left_wheel_link"/>
-    <axis xyz="0 1 0"/>
-  </joint>
-  <link name="right_wheel_link">
-    <inertial>
-      <origin xyz="0 0 0"/>
-      <mass value="0.01" />
-      <inertia ixx="0.001" ixy="0.0" ixz="0.0"
-        iyy="0.001" iyz="0.0" izz="0.001" />
-    </inertial>
-    <visual>
-      <origin xyz="0 0 0" rpy="0 1.5707 1.5707" />
-      <geometry>
-        <cylinder radius="0.033" length = "0.023"/>
-      </geometry>
-    </visual>
-    <collision>
-      <origin xyz="0 0 0" rpy="0 1.5707 1.5707" />
-      <geometry>
-        <cylinder radius="0.033" length = "0.023"/>
-      </geometry>
-    </collision>
-  </link>
-  <joint name="right_wheel_joint" type="continuous">
-    <origin xyz="0 -0.13 0.015" rpy="0 0 0"/>
-    <parent link="base_link"/>
-    <child link="right_wheel_link"/>
-    <axis xyz="0 1 0"/>
-  </joint>
-  <link name="rear_wheel_link">
-    <inertial>
-      <origin xyz="0 0 0"/>
-      <mass value="0.001" />
-      <inertia ixx="0.0001" ixy="0.0" ixz="0.0"
-        iyy="0.0001" iyz="0.0" izz="0.0001" />
-    </inertial>
-    <visual>
-      <origin xyz="0 0 0" rpy="0 1.5707 1.5707"/>
-      <geometry>
-        <sphere radius="0.015" />
-      </geometry>
-    </visual>
-    <collision>
-      <origin xyz="0 0 0" rpy="0 1.5707 1.5707" />
-      <geometry>
-        <sphere radius="0.015" />
-      </geometry>
-    </collision>
-  </link>
-  <!-- fixed because there's no transmission -->
-  <joint name="rear_castor_joint" type="fixed">
-    <origin xyz="-0.13 0 0.0" rpy="0 0 0"/>
-    <parent link="base_link"/>
-    <child link="rear_wheel_link"/>
-    <axis xyz="0 1 0"/>
-  </joint>
-  <link name="front_wheel_link">
-    <inertial>
-      <origin xyz="0 0 0" />
-      <mass value="0.01" />
-      <inertia ixx="0.001" ixy="0.0" ixz="0.0"
-        iyy="0.001" iyz="0.0" izz="0.001" />
-    </inertial>
-    <visual>
-      <origin xyz="0 0 0" rpy="0 1.5707 1.5707"/>
-      <geometry>
-        <sphere radius="0.018" />
-      </geometry>
-    </visual>
-    <collision>
-      <origin xyz="0 0 0" rpy="0 1.5707 1.5707" />
-      <geometry>
-        <sphere radius="0.018" />
-      </geometry>
-    </collision>
-  </link>
-  <!-- fixed because there's no transmission -->
-  <joint name="front_castor_joint" type="fixed">
-    <origin xyz="0.13 0 0.0" rpy="0 0 0"/>
-    <parent link="base_link"/>
-    <child link="front_wheel_link"/>
-    <axis xyz="0 1 0"/>
-  </joint>
-  <joint name="gyro_joint" type="fixed">
-    <axis xyz="0 1 0" />
-    <origin xyz="0 0 0.04" rpy="0 0 0" />
-    <parent link="base_link"/>
-    <child link="gyro_link"/>
-  </joint>
-  <link name="gyro_link">
-    <inertial>
-      <mass value="0.001" />
-      <origin xyz="0 0 0" rpy="0 0 0" />
-      <inertia ixx="0.0001" ixy="0" ixz="0" iyy="0.000001" iyz="0" izz="0.0001" />
-    </inertial>
-  </link>
-  <joint name="laser_joint" type="fixed">
-    <origin xyz="-0.065 0 0.075" rpy="0 0 0" />
-    <parent link="base_link" />
-    <child link="laser" />
-  </joint>
-  <link name="laser">
-    <visual>
-      <geometry>
-        <box size="0.02 0.035 0.002" />
-      </geometry>
-      <material name="Green" />
-    </visual>
-    <inertial>
-      <mass value="0.001" />
-      <origin xyz="0 0 0" />
-      <inertia ixx="0.0001" ixy="0.0" ixz="0.0"
-        iyy="0.0001" iyz="0.0"
-        izz="0.0001" />
-    </inertial>
-  </link>
-  <!-- Simulation sensors -->
-  <turtlebot_sim_imu/>
-  <turtlebot_sim_laser/>
-  <turtlebot_sim_create/>
-  <turtlebot_sim_wall_sensors/>
+	  <xacro:macro name="create">
+	    <material name="Green">
+	      <color rgba="0.0 0.8 0.0 1.0"/>
+	    </material>
+	  <!-- base_footprint is a fictitious link(frame) that is on the ground right below base_link origin, navigation stack depends on this frame -->
+	  <link name="base_footprint">
+	<!--
+	    <inertial>
+	      <mass value="0.0001" />
+	      <origin xyz="0 0 0" />
+	      <inertia ixx="0.0001" ixy="0.0" ixz="0.0"
+	              iyy="0.0001" iyz="0.0"
+	              izz="0.0001" />
+	    </inertial>
+	-->
+	    <visual>
+	      <origin xyz="0 0 0" rpy="0 0 0" />
+	      <geometry>
+	        <box size="0.001 0.001 0.001" />
+	      </geometry>
+	      <material name="Green" />
+	    </visual>
+	    <collision>
+	      <origin xyz="0 0 0.017" rpy="0 0 0" />
+	      <geometry>
+	       <box size="0.001 0.001 0.001" />
+	      </geometry>
+	    </collision>
+	  </link>
+	  <link name="base_link">
+	    <inertial>
+	      <mass value="2" />
+	      <origin xyz="0 0 0.0" />
+	      <inertia ixx="0.01" ixy="0.0" ixz="0.0"
+	        iyy="0.01" iyz="0.0" izz="0.5" />
+	    </inertial>
+	    <visual>
+	      <origin xyz=" 0 0 0.0308" rpy="0 0 0" />
+	      <geometry>
+	        <mesh filename="package://create_description/meshes/create_body.dae"/>
+	      </geometry>
+	    </visual>
+	    <collision>
+	      <origin xyz="0.0 0.0 0.0308" rpy="0 0 0" />
+	      <geometry>
+	        <cylinder length="0.0611632" radius="0.016495"/>
+	      </geometry>
+	    </collision>
+	  </link>
+	  <link name="wall_sensor_link">
+	    <inertial>
+	      <mass value="0.01" />
+	      <origin xyz="0 0 0"/>
+	      <inertia ixx="0.001" ixy="0.0" ixz="0.0"
+	        iyy="0.001" iyz="0.0" izz="0.001" />
+	    </inertial>
+	  </link>
+	  <link name="left_cliff_sensor_link">
+	    <inertial>
+	      <mass value="0.01" />
+	      <origin xyz="0 0 0"/>
+	      <inertia ixx="0.001" ixy="0.0" ixz="0.0"
+	        iyy="0.001" iyz="0.0" izz="0.001" />
+	    </inertial>
+	  </link>
+	  <link name="right_cliff_sensor_link">
+	    <inertial>
+	      <mass value="0.01" />
+	      <origin xyz="0 0 0"/>
+	      <inertia ixx="0.001" ixy="0.0" ixz="0.0"
+	        iyy="0.001" iyz="0.0" izz="0.001" />
+	    </inertial>
+	  </link>
+	  <link name="leftfront_cliff_sensor_link">
+	    <inertial>
+	      <mass value="0.01" />
+	      <origin xyz="0 0 0"/>
+	      <inertia ixx="1.0" ixy="0.0" ixz="0.0"
+	        iyy="0.01" iyz="0.0" izz="0.01" />
+	    </inertial>
+	  </link>
+	  <link name="rightfront_cliff_sensor_link">
+	    <inertial>
+	      <mass value="0.01" />
+	      <origin xyz="0 0 0"/>
+	      <inertia ixx="0.001" ixy="0.0" ixz="0.0"
+	        iyy="0.001" iyz="0.0" izz="0.001" />
+	    </inertial>
+	  </link>
+	  <joint name="base_footprint_joint" type="fixed">
+	    <origin xyz="0 0 0.017" rpy="0 0 0" />
+	    <parent link="base_footprint"/>
+	    <child link="base_link" />
+	  </joint>
+	  <joint name="base_wall_sensor_joint" type="fixed">
+	    <origin xyz="0.09 -0.120 0.042" rpy="0 0 -1.0" />
+	    <parent link="base_link"/>
+	    <child link="wall_sensor_link" />
+	  </joint>
+	  <joint name="base_left_cliff_sensor_joint" type="fixed">
+	    <origin xyz="0.07 0.14 0.01" rpy="0 1.57079 0" />
+	    <parent link="base_link"/>
+	    <child link="left_cliff_sensor_link" />
+	  </joint>
+	  <joint name="base_right_cliff_sensor_joint" type="fixed">
+	    <origin xyz="0.07 -0.14 0.01" rpy="0 1.57079 0" />
+	    <parent link="base_link"/>
+	    <child link="right_cliff_sensor_link" />
+	  </joint>
+	  <joint name="base_leftfront_cliff_sensor_joint" type="fixed">
+	    <origin xyz="0.15 0.04 0.01" rpy="0 1.57079 0" />
+	    <parent link="base_link"/>
+	    <child link="leftfront_cliff_sensor_link" />
+	  </joint>
+	  <joint name="base_rightfront_cliff_sensor_joint" type="fixed">
+	    <origin xyz="0.15 -0.04 0.01" rpy="0 1.57079 0" />
+	    <parent link="base_link"/>
+	    <child link="rightfront_cliff_sensor_link" />
+	  </joint>
+	  <link name="left_wheel_link">
+	    <inertial>
+	      <origin xyz="0 0 0"/>
+	      <mass value="0.01" />
+	      <inertia ixx="0.001" ixy="0.0" ixz="0.0"
+	        iyy="0.001" iyz="0.0" izz="0.001" />
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
Commit message: fixes broken create visualisation * removes scaling * corrects unit in collada mesh

File: create_description/urdf/create.urdf.xacro (robot description, xacro)
@@ -6,6 +6,4 @@
   <!-- Macro for TurtleBot body. Including Gazebo extensions, but does not include Kinect -->
   <include filename="$(find create_description)/urdf/create_gazebo.urdf.xacro"/>
-  <property name="base_x" value="0.33" />
-  <property name="base_y" value="0.33" />
 	  <xacro:macro name="create">
 	    <material name="Green">
@@ -14,13 +12,4 @@
 	  <!-- base_footprint is a fictitious link(frame) that is on the ground right below base_link origin, navigation stack depends on this frame -->
 	  <link name="base_footprint">
-	<!--
-	    <inertial>
-	      <mass value="0.0001" />
-	      <origin xyz="0 0 0" />
-	      <inertia ixx="0.0001" ixy="0.0" ixz="0.0"
-	              iyy="0.0001" iyz="0.0"
-	              izz="0.0001" />
-	    </inertial>
-	-->
 	    <visual>
 	      <origin xyz="0 0 0" rpy="0 0 0" />

Commit message: removes laser simulation (fixes #11)

File: create_description/urdf/create.urdf.xacro (robot description, xacro)
@@ -259,5 +259,4 @@
 	  <sim_create_cliff_sensors/>
     <sim_imu/>
-	  <sim_laser/>
   </xacro:macro>
 </robot>

File: create_description/urdf/create_gazebo.urdf.xacro (robot description, xacro)
@@ -177,35 +177,3 @@
 	  </gazebo>
 	</xacro:macro>
-	<xacro:macro name="sim_laser">
-	  <gazebo reference="laser">
-      <sensor type="ray" name="laser">
-        <always_on>true</always_on>
-        <update_rate>20.0</update_rate>
-        <pose>0 0 0 0 0 0</pose>
-        <visualize>false</visualize>
-        <ray>
-          <scan>
-            <horizontal>
-              <samples>180</samples>
-              <resolution>1</resolution>
-              <min_angle>${-130.0*M_PI/180.0}</min_angle>
-              <max_angle>${130.0*M_PI/180.0}</max_angle>
-            </horizontal>
-          </scan>
-          <range>
-            <min>0.08</min>
-            <max>10.0</max>
-            <resolution>0.01</resolution>
-          </range>
-        </ray>
-        <plugin name="gazebo_ros_laser_controller" filename="libgazebo_ros_laser.so">
-          <gaussianNoise>0.005</gaussianNoise>
-          <alwaysOn>true</alwaysOn>
-          <updateRate>20</updateRate>
-          <topicName>scan</topicName>
-          <frameName>laser</frameName>
-        </plugin>
-      </sensor>
-	  </gazebo>
-  </xacro:macro>
 </robot>

Commit message: update xacro:property tag usage to stricter standard

File: create_description/urdf/create.urdf.xacro (robot description, xacro)
@@ -3,6 +3,6 @@
   <!-- Macro for TurtleBot body. Including Gazebo extensions, but does not include Kinect -->
   <xacro:include filename="$(find create_description)/urdf/create_gazebo.urdf.xacro"/>
-  <property name="base_x" value="0.33" />
-  <property name="base_y" value="0.33" />
+  <xacro:property name="base_x" value="0.33" />
+  <xacro:property name="base_y" value="0.33" />
 	  <xacro:macro name="create">
 	    <material name="Green">
